File: schematic/schematics.kicad_sch (KiCad schematic)
At the start: 24 parts, among them J2 To garage door opener main pcb, J3 To encoder, Q1 BC547, Q2 BC547, U1 AHT20, U2 BMP280, U3 PC817, U4 PC817

Commit message: Use same pin for encoder and pulse counter
Connections:
- net at A1.23 (I35), R1.1, R6.2: no longer A1.2 (IO36)
Changed lines of the file:
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@@
   (junction (at 168.91 73.66) (diameter 0) (color 0 0 0 0)
   )
-  (junction (at 148.59 110.49) (diameter 0) (color 0 0 0 0)
-  )
   (wire (pts (xy 208.28 119.38) (xy 208.28 129.54))
     (stroke (width 0) (type default))
@@
     (stroke (width 0) (type default))
   )
-  (wire (pts (xy 148.59 78.74) (xy 148.59 110.49))
-    (stroke (width 0) (type default))
-  )
   (wire (pts (xy 100.33 57.15) (xy 110.49 57.15))
     (stroke (width 0) (type default))
@@
     (stroke (width 0) (type default))
   )
-  (wire (pts (xy 100.33 95.25) (xy 97.79 95.25))
-    (stroke (width 0) (type default))
-  )
   (wire (pts (xy 224.79 135.89) (xy 222.25 135.89))
     (stroke (width 0) (type default))
@@
     (stroke (width 0) (type default))
   )
-  (wire (pts (xy 97.79 78.74) (xy 148.59 78.74))
-    (stroke (width 0) (type default))
-  )
   (wire (pts (xy 209.55 116.84) (xy 207.01 116.84))
     (stroke (width 0) (type default))
@@
     (stroke (width 0) (type default))
   )
-  (wire (pts (xy 97.79 95.25) (xy 97.79 78.74))
-    (stroke (width 0) (type default))
-  )
   (wire (pts (xy 195.58 49.53) (xy 195.58 53.34))
     (stroke (width 0) (type default))
@@
     (stroke (width 0) (type default))
   )
-  (wire (pts (xy 148.59 110.49) (xy 158.75 110.49))
-    (stroke (width 0) (type default))
-  )
-  (wire (pts (xy 138.43 110.49) (xy 148.59 110.49))
-    (stroke (width 0) (type default))
-  )
+  (wire (pts (xy 138.43 110.49) (xy 158.75 110.49))
+    (stroke (width 0) (type default))
+  )
